Commit message: camera calibration medium

File: ros2_ws/src/manipulators/assets/robots/kinova/urdf/gen3_2f85.urdf (robot description, URDF)
Before this commit: robot gen3_, 20 links, 19 joints
Links:
- added link gen3_end_link
Joints:
- removed joint gen3_end_effector
- added joint gen3_end_effector_joint: type fixed, parent gen3_end_link, child gen3_end_effector_link, origin xyz=0 0 0.15 rpy=0 0 0, axis 0 0 0
- added joint gen3_end_joint: type fixed, parent gen3_bracelet_link, child gen3_end_link, origin xyz=0 0 -0.0615250000000001 rpy=3.14159265358979 1.09937075168372E-32 0, axis 0 0 0
- joint gen3_robotiq_85_base_joint: parent gen3_end_effector_link -> gen3_end_link
